File: power system.sch (EAGLE design)
At the start: 43 parts

Commit message: 1. increase the wire width 2. merge the two brd file 3. change the fuse value and connector order 4. approve the DRC error
Parts:
- F2, F3: value 3A -> 4A
- F4: value 4A -> 2A
Connections:
- net N$12: now also M_Y-1.S; no longer M_DC-1.S
- net N$6: now also M_DC-1.S; no longer M_Y-1.S
Other:
- moved on the sheet: M_DC-1, M_DC-2, M_Y-1, M_Y-2
Changed lines of the file:
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@@
 <part name="GND13" library="supply1" deviceset="GND" device=""/>
 <part name="F1" library="fuse" deviceset="TE5" device="" value="2A"/>
-<part name="F2" library="fuse" deviceset="TE5" device="" value="3A"/>
-<part name="F3" library="fuse" deviceset="TE5" device="" value="3A"/>
-<part name="F4" library="fuse" deviceset="TE5" device="" value="4A"/>
+<part name="F2" library="fuse" deviceset="TE5" device="" value="4A"/>
+<part name="F3" library="fuse" deviceset="TE5" device="" value="4A"/>
+<part name="F4" library="fuse" deviceset="TE5" device="" value="2A"/>
 <part name="F5" library="fuse" deviceset="TE5" device="" value="2A"/>
 <part name="F6" library="fuse" deviceset="TE5" device="" value="2A"/>
@@
 <part name="GND16" library="supply1" deviceset="GND" device=""/>
 <part name="M_X" library="con-molex" deviceset="5566-2" device=""/>
+<part name="M_DC" library="con-molex" deviceset="5566-2" device=""/>
 <part name="M_Y" library="con-molex" deviceset="5566-2" device=""/>
-<part name="M_DC" library="con-molex" deviceset="5566-2" device=""/>
 <part name="M_R" library="con-molex" deviceset="5566-2" device=""/>
 <part name="12V1" library="con-molex" deviceset="5566-2" device=""/>
@@
 <instance part="M_X" gate="-1" x="127" y="116.84"/>
 <instance part="M_X" gate="-2" x="127" y="111.76"/>
-<instance part="M_Y" gate="-1" x="127" y="101.6"/>
-<instance part="M_Y" gate="-2" x="127" y="96.52"/>
-<instance part="M_DC" gate="-1" x="127" y="83.82"/>
-<instance part="M_DC" gate="-2" x="127" y="78.74"/>
+<instance part="M_DC" gate="-1" x="127" y="101.6"/>
+<instance part="M_DC" gate="-2" x="127" y="96.52"/>
+<instance part="M_Y" gate="-1" x="127" y="83.82"/>
+<instance part="M_Y" gate="-2" x="127" y="78.74"/>
 <instance part="M_R" gate="-1" x="127" y="66.04"/>
 <instance part="M_R" gate="-2" x="127" y="60.96"/>
@@
 <wire x1="104.14" y1="91.44" x2="124.46" y2="91.44" width="0.1524" layer="91"/>
 <junction x="104.14" y="91.44"/>
-<pinref part="M_Y" gate="-2" pin="S"/>
+<pinref part="M_DC" gate="-2" pin="S"/>
 <wire x1="124.46" y1="91.44" x2="124.46" y2="96.52" width="0.1524" layer="91"/>
 </segment>
@@
 <wire x1="104.14" y1="73.66" x2="124.46" y2="73.66" width="0.1524" layer="91"/>
 <junction x="104.14" y="73.66"/>
-<pinref part="M_DC" gate="-2" pin="S"/>
+<pinref part="M_Y" gate="-2" pin="S"/>
 <wire x1="124.46" y1="73.66" x2="124.46" y2="78.74" width="0.1524" layer="91"/>
 </segment>
@@
 <wire x1="104.14" y1="101.6" x2="124.46" y2="101.6" width="0.1524" layer="91"/>
 <junction x="104.14" y="101.6"/>
-<pinref part="M_Y" gate="-1" pin="S"/>
+<pinref part="M_DC" gate="-1" pin="S"/>
 </segment>
 </net>
@@
 <wire x1="104.14" y1="83.82" x2="124.46" y2="83.82" width="0.1524" layer="91"/>
 <junction x="104.14" y="83.82"/>
-<pinref part="M_DC" gate="-1" pin="S"/>
+<pinref part="M_Y" gate="-1" pin="S"/>
 </segment>
 </net>
@@
 </sheet>
 </sheets>
+<errors>
+</errors>
 </schematic>
 </drawing>
